Commit message: fix(ur5e): define default values for urdf parameters

File: ros/ur5e_catkin_ws/src/coarobo_teleop/description/onrobot_qc_r_v3/urdf/onrobot_qc_r_v3.xacro (robot description, xacro)
@@ -11,10 +11,10 @@
     <visual>
       <geometry>
-        <mesh filename="package://coarobo_teleop/description/onrobot_qc_r_v3/meshes/visual/qc_r_v3.stl"/>
+        <mesh filename="package://coarobo_teleop/description/onrobot_qc_r_v3/meshes/visual/onrobot_qc_r_v3.stl"/>
       </geometry>
     </visual>
     <collision>
       <geometry>
-        <mesh filename="package://coarobo_teleop/description/onrobot_qc_r_v3/meshes/collision/qc_r_v3.stl"/>
+        <mesh filename="package://coarobo_teleop/description/onrobot_qc_r_v3/meshes/collision/onrobot_qc_r_v3.stl"/>
       </geometry>
     </collision>

File: ros/ur5e_catkin_ws/src/coarobo_teleop/urdf/ur5e_rg2_gazebo.xacro (robot description, xacro)
@@ -8,8 +8,8 @@
   <xacro:arg name="use_nominal_extrinsics" default="true" />
   <xacro:arg name="robot_model" default="ur5e"/>
-  <xacro:arg name="joint_limit_params" default=""/>
-  <xacro:arg name="physical_params" default=""/>
-  <xacro:arg name="kinematics_params" default=""/>
-  <xacro:arg name="visual_params" default=""/>
+  <xacro:arg name="joint_limit_params" default="$(find ur_description)/config/ur5e/joint_limits.yaml"/>
+  <xacro:arg name="physical_params" default="$(find ur_description)/config/ur5e/physical_parameters.yaml"/>
+  <xacro:arg name="kinematics_params" default="$(find ur_description)/config/ur5e/default_kinematics.yaml"/>
+  <xacro:arg name="visual_params" default="$(find ur_description)/config/ur5e/visual_parameters.yaml"/>
   <xacro:arg name="transmission_hw_interface" default="hardware_interface/EffortJointInterface"/>
   <xacro:arg name="safety_limits" default="false"/>
@@ -52,10 +52,10 @@
   <xacro:onrobot_qc_r_v3 parent="camera_adapter_link">
     <!-- Rotate 180 degrees so the gripper faces outwards instead of into the mount -->
-    <origin xyz="0 0 0" rpy="0 3.14159 0" />
+    <origin xyz="0 0 -0.0125" rpy="0 3.14159 0" />
   </xacro:onrobot_qc_r_v3>
   <joint name="qc_tool_mount-onrobot_rg2_base" type="fixed">
     <parent link="qc_tool_mount" />
     <child link="onrobot_rg2_base_link" />
-    <origin xyz="0 0 0" rpy="0 0 0" />
+    <origin xyz="0 0 -0.005" rpy="0 0 -1.5708" />
     <axis xyz="0 0 1" />
   </joint>
@@ -96,5 +96,5 @@
   <xacro:sensor_d435i parent="camera_mount_link" name="wrist_camera" use_nominal_extrinsics="$(arg use_nominal_extrinsics)">
     <!-- Subtracted 8 degrees (0.139626 radians) to the pitch axis -->
-    <origin xyz="0.0 -0.095 -0.011" rpy="0 ${-1.5708 - 0.139626} -1.5708"/>
+    <origin xyz="0.0 -0.075 -0.011" rpy="0 ${1.5708 - 0.139626} -1.5708"/>
   </xacro:sensor_d435i>
 </robot>
