Commit message: refactor(ur5e): rename UR5e package and config files for better separation of functions

File: ros/ur5e_catkin_ws/src/sde_ur5e_launch/description/onrobot_quick_changer_qc-r_v3/urdf/onrobot_quick_changer_qc-r_v3.xacro (robot description, xacro)
@@ -11,10 +11,10 @@
     <visual>
       <geometry>
-        <mesh filename="package://coarobo_teleop/description/onrobot_qc_r_v3/meshes/visual/onrobot_qc_r_v3.stl"/>
+        <mesh filename="package://sde_ur5e_launch/description/onrobot_quick_changer_qc-r_v3/meshes/visual/onrobot_quick_changer_qc-r_v3.stl"/>
       </geometry>
     </visual>
     <collision>
       <geometry>
-        <mesh filename="package://coarobo_teleop/description/onrobot_qc_r_v3/meshes/collision/onrobot_qc_r_v3.stl"/>
+        <mesh filename="package://sde_ur5e_launch/description/onrobot_quick_changer_qc-r_v3/meshes/collision/onrobot_quick_changer_qc-r_v3.stl"/>
       </geometry>
     </collision>

File: ros/ur5e_catkin_ws/src/sde_ur5e_launch/description/picknik_ur5_realsense_camera_adapter/urdf/picknik_ur5_realsense_camera_adapter.xacro (robot description, xacro)
@@ -19,5 +19,5 @@
         <origin xyz="0 0 0" rpy="0 0 0" />
         <geometry>
-          <mesh filename="package://coarobo_teleop/description/picknik_ur5_realsense_camera_adapter/meshes/picknik_ur5_realsense_camera_adapter.STL" scale="1 1 1" />
+          <mesh filename="package://sde_ur5e_launch/description/picknik_ur5_realsense_camera_adapter/meshes/picknik_ur5_realsense_camera_adapter.stl" scale="1 1 1" />
         </geometry>
         <material name="dark_grey">
@@ -28,5 +28,5 @@
         <origin xyz="0 0 0" rpy="0 0 0" />
         <geometry>
-          <mesh filename="package://coarobo_teleop/description/picknik_ur5_realsense_camera_adapter/meshes/picknik_ur5_realsense_camera_adapter.STL" scale="1 1 1" />
+          <mesh filename="package://sde_ur5e_launch/description/picknik_ur5_realsense_camera_adapter/meshes/picknik_ur5_realsense_camera_adapter.stl" scale="1 1 1" />
         </geometry>
       </collision>

File: ros/ur5e_catkin_ws/src/sde_ur5e_launch/urdf/ur5e_gazebo.xacro (robot description, xacro)
@@ -4,6 +4,6 @@
   <xacro:include filename="$(find onrobot_rg_description)/urdf/onrobot_rg2_model_macro.xacro"/>
   <xacro:include filename="$(find realsense2_description)/urdf/_d435i.urdf.xacro"/>
-  <xacro:include filename="$(find coarobo_teleop)/description/picknik_ur5_realsense_camera_adapter/urdf/picknik_ur5_realsense_camera_adapter.xacro"/>
-  <xacro:include filename="$(find coarobo_teleop)/description/onrobot_qc_r_v3/urdf/onrobot_qc_r_v3.xacro"/>
+  <xacro:include filename="$(find sde_ur5e_launch)/description/picknik_ur5_realsense_camera_adapter/urdf/picknik_ur5_realsense_camera_adapter.xacro"/>
+  <xacro:include filename="$(find sde_ur5e_launch)/description/onrobot_quick_changer_qc-r_v3/urdf/onrobot_quick_changer_qc-r_v3.xacro"/>
   <xacro:arg name="use_nominal_extrinsics" default="true" />
   <xacro:arg name="robot_model" default="ur5e"/>
@@ -90,7 +90,8 @@
   </xacro:picknik_camera_adapter>
   <!-- External RealSense D435i Camera (Environment view, using world as parent) -->
-  <xacro:sensor_d435i parent="world" name="external_camera" use_nominal_extrinsics="$(arg use_nominal_extrinsics)">
+  <!-- TODO: Uncomment and tune the origin once the external camera mount position is known. -->
+  <!-- <xacro:sensor_d435i parent="world" name="external_camera" use_nominal_extrinsics="$(arg use_nominal_extrinsics)">
     <origin xyz="1.0 0.0 1.0" rpy="0 0.5 3.14159"/>
-  </xacro:sensor_d435i>
+  </xacro:sensor_d435i> -->
   <!-- Wrist-mounted RealSense D435i Camera (Attached to the PickNik adapter's mount link) -->
   <xacro:sensor_d435i parent="camera_mount_link" name="wrist_camera" use_nominal_extrinsics="$(arg use_nominal_extrinsics)">

Commit message: refactor(ur5e): add real-world configuration/model/description for UR5e robot

File: ros/ur5e_catkin_ws/src/sde_ur5e_launch/description/onrobot_quick_changer_qc-r_v3/urdf/onrobot_quick_changer_qc-r_v3.xacro (robot description, xacro)
@@ -13,4 +13,7 @@
         <mesh filename="package://sde_ur5e_launch/description/onrobot_quick_changer_qc-r_v3/meshes/visual/onrobot_quick_changer_qc-r_v3.stl"/>
       </geometry>
+      <material name="qc_blue">
+        <color rgba="0 0.35 0.8 1"/>
+      </material>
     </visual>
     <collision>
