Commit message: refactor(ur5e) : improve urdf

File: ros/ur5e_catkin_ws/src/sde_ur5e_launch/urdf/ur5e_realworld.xacro (robot description, xacro)
@@ -27,42 +27,25 @@
     safety_k_position="$(arg safety_k_position)"
   />
-  <link name="onrobot_rg2_base_link">
-    <inertial>
-      <origin xyz="0.0 0.0 0.0" rpy="0 0 0" />
-      <mass value="0.7" />
-      <inertia ixx="1.0E-03" ixy="1.0E-06" ixz="1.0E-06" iyy="1.0E-03" iyz="1.0E-06" izz="1.0E-03" />
-    </inertial>
-    <visual>
-      <origin xyz="0 0 0" rpy="0 0 0" />
-      <geometry>
-        <mesh filename="package://onrobot_rg_description/meshes/rg2/visual/base_link.stl" />
-      </geometry>
-      <material name="">
-        <color rgba="0.8 0.8 0.8 1" />
-      </material>
-    </visual>
-    <collision>
-      <origin xyz="0 0 0" rpy="0 0 0" />
-      <geometry>
-        <mesh filename="package://onrobot_rg_description/meshes/rg2/collision/base_link.stl" />
-      </geometry>
-    </collision>
-  </link>
-  <!-- Instantiate the QC using its new macro, attached to the adapter -->
-  <xacro:onrobot_qc_r_v3 parent="camera_adapter_link">
-    <!-- Rotate 180 degrees so the gripper faces outwards instead of into the mount -->
-    <origin xyz="0 0 -0.0125" rpy="0 3.14159 0" />
-  </xacro:onrobot_qc_r_v3>
+  <!-- Instantiate gripper -->
+  <xacro:onrobot_rg2 prefix=""/>
+  <!-- Attach gripper to quick changer -->
   <joint name="qc_tool_mount-onrobot_rg2_base" type="fixed">
     <parent link="qc_tool_mount" />
     <child link="onrobot_rg2_base_link" />
-    <origin xyz="0 0 -0.005" rpy="0 0 -1.5708" />
+    <origin xyz="0 0 -0.007" rpy="0 0 -1.5708" />
     <axis xyz="0 0 1" />
   </joint>
-  <xacro:finger_links prefix="" fingerprefix="left"/>
-  <xacro:finger_links prefix="" fingerprefix="right"/>
-  <xacro:finger_joint prefix=""/>
-  <xacro:right_outer_knuckle_joint prefix=""/>
+  <!-- Quick changer attached to the camera adapter -->
+  <xacro:onrobot_qc_r_v3 parent="camera_adapter_link">
+    <!-- Rotate 180 degrees so the gripper faces outwards instead of into the mount -->
+    <origin xyz="0 0 0.01" rpy="0 0 0" />
+  </xacro:onrobot_qc_r_v3>
+  <!-- Camera Adapter (Attached to Robot's flange/tool0) -->
+  <xacro:picknik_camera_adapter parent="tool0">
+    <!-- Fine-tune this origin based on how the adapter sits on the flange -->
+    <origin xyz="0.0 0.0 -0.001" rpy="0 0 0"/>
+  </xacro:picknik_camera_adapter>
   <link name="world"/>
+  <!-- Robot base is attached to the world (fixed joint)  -->
   <joint name="world_joint" type="fixed">
     <parent link="world"/>
@@ -76,9 +59,4 @@
     <origin xyz="0 0 0" rpy="0 0 0"/>
   </joint>
-  <!-- PickNik Camera Adapter (Attached to Robot's flange/tool0) -->
-  <xacro:picknik_camera_adapter parent="tool0">
-    <!-- Fine-tune this origin based on how the adapter sits on the flange -->
-    <origin xyz="0.0 0.0 0.01" rpy="0 3.14159 0"/>
-  </xacro:picknik_camera_adapter>
   <!-- External RealSense D435i Camera (Environment view, using world as parent) -->
   <!-- TODO: Uncomment and tune the origin once the external camera mount position is known. -->
@@ -89,5 +67,5 @@
   <xacro:sensor_d435i parent="camera_mount_link" name="wrist_camera" use_nominal_extrinsics="$(arg use_nominal_extrinsics)">
     <!-- Subtracted 8 degrees (0.139626 radians) to the pitch axis -->
-    <origin xyz="0.0 -0.075 -0.011" rpy="0 ${1.5708 - 0.139626} -1.5708"/>
+    <origin xyz="0 -0.065 0.016" rpy="3.14159 ${3.14159 + 1.5708 - 0.139626} -1.5708"/>
   </xacro:sensor_d435i>
 </robot>

Commit message: refactor(ur5e) : set demo  parameters

File: ros/ur5e_catkin_ws/src/sde_ur5e_launch/urdf/ur5e_realworld.xacro (robot description, xacro)
@@ -62,5 +62,5 @@
   <!-- TODO: Uncomment and tune the origin once the external camera mount position is known. -->
   <xacro:sensor_d435i parent="world" name="external_camera" use_nominal_extrinsics="$(arg use_nominal_extrinsics)">
-    <origin xyz="1.0 0.0 1.0" rpy="0 0.5 3.14159"/>
+    <origin xyz="-1.5 0.3 0.3" rpy="0 0 0"/>
   </xacro:sensor_d435i>
   <!-- Wrist-mounted RealSense D435i Camera (Attached to the PickNik adapter's mount link) -->

Commit message: refactor(ur5e) : fix security velocity issue and update urdf for demo

File: ros/ur5e_catkin_ws/src/sde_ur5e_launch/urdf/ur5e_realworld.xacro (robot description, xacro)
@@ -62,5 +62,5 @@
   <!-- TODO: Uncomment and tune the origin once the external camera mount position is known. -->
   <xacro:sensor_d435i parent="world" name="external_camera" use_nominal_extrinsics="$(arg use_nominal_extrinsics)">
-    <origin xyz="-1.5 0.3 0.3" rpy="0 0 0"/>
+    <origin xyz="0 -0.254 0.38" rpy="0 0.31 ${3.14159 - 0.54}"/>
   </xacro:sensor_d435i>
   <!-- Wrist-mounted RealSense D435i Camera (Attached to the PickNik adapter's mount link) -->
